Commit message: change initial position, added color, checked the maximum spawn locations, changed the table setting, start of teleoperation data

File: assets/F14_URDF_rev_2_0_1 2/urdf/FlaminGO_14Dof_Arm_Robot_v2.urdf (robot description, URDF)
Before this commit: robot FlaminGO_14Dof_Arm_Robot_v2, 19 links, 18 joints
Links:
- link base_link: geometry collision mesh filename=package://FlaminGO_14Dof_Arm_Robot_v2/meshes/base_link.STL; visual mesh filename=package://FlaminGO_14Dof_Arm_Robot_v2/meshes/base_link_pill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
